Commit message: Adding the base for collision

File: ros2_kortex/kortex_description/robots/gen3.xacro (robot description, xacro)
@@ -3,5 +3,5 @@
     <!-- Arguments -->
     <xacro:arg name="arm" default="gen3" />
-    <xacro:arg name="dof" default="" />
+    <xacro:arg name="dof" default="7" />
     <xacro:arg name="vision" default="false" />
     <xacro:arg name="robot_ip" default="192.168.11.11" />
@@ -12,5 +12,5 @@
     <xacro:arg name="session_inactivity_timeout_ms" default="60000" />
     <xacro:arg name="connection_inactivity_timeout_ms" default="2000" />
-    <xacro:arg name="gripper" default="" />
+    <xacro:arg name="gripper" default="robotiq_2f_85" />
     <xacro:arg name="gripper_joint_name" default="finger_joint" />
     <xacro:arg name="gripper_max_velocity" default="100.0" />
@@ -29,5 +29,26 @@
     <!-- convert to property to use substitution in function -->
     <xacro:property name="initial_positions_file" default="$(arg initial_positions_file)"/>
-    <link name="world" />
+    <link name="world">
+      <!-- Inertial properties -->
+      <inertial>
+        <origin xyz="0 0 0" rpy="0 0 0" />
+        <mass value="1.0" /> <!-- Adjust mass as needed -->
+        <inertia ixx="0.1" ixy="0.0" ixz="0.0" iyy="0.1" iyz="0.0" izz="0.1" />
+      </inertial>
+      <!-- Visual properties -->
+      <visual>
+        <origin xyz="0 0 0" rpy="0 0 0" />
+        <geometry>
+          <box size="2 1 0.2" />
+        </geometry>
+      </visual>
+      <!-- Collision properties -->
+      <collision>
+        <origin xyz="0 0 0" rpy="0 0 0" />
+        <geometry>
+          <box size="2 1 0.2" />
+        </geometry>
+      </collision>
+    </link>
     <xacro:load_robot
         parent="world"

File: ros2_kortex/kortex_description/robots/kinova.urdf.xacro (robot description, xacro)
@@ -38,5 +38,24 @@
   <xacro:property name="initial_positions_file" default="$(arg initial_positions_file)"/>
   <!-- create link fixed to the "world" -->
-  <link name="world" />
+    <!-- World link -->
+  <link name="world">
+    <inertial>
+      <origin xyz="0 0 0" rpy="0 0 0" />
+      <mass value="1.0" />
+      <inertia ixx="0.1" ixy="0.0" ixz="0.0" iyy="0.1" iyz="0.0" izz="0.1" />
+    </inertial>
+    <visual>
+      <origin xyz="0 0 0" rpy="0 0 0" />
+      <geometry>
+        <box size="2 1 0.2" />
+      </geometry>
+    </visual>
+    <collision>
+      <origin xyz="0 0 0" rpy="0 0 0" />
+      <geometry>
+        <box size="2 1 0.2" />
+      </geometry>
+    </collision>
+  </link>
   <xacro:load_robot
     parent="world"

File: ros2_kortex/kortex_description/robots/kortex_robot.xacro (robot description, xacro)
@@ -32,5 +32,6 @@
     moveit_active:=false">
     <!-- Include and load arm macro files -->
-    <xacro:include filename="$(find kortex_description)/arms/${arm}/${dof}dof/urdf/${arm}_macro.xacro" />
+    <!--xacro:include filename="$(find kortex_description)/arms/${arm}/${dof}dof/urdf/${arm}_macro.xacro" /-->
+    <xacro:include filename="$(find kortex_description)/arms/gen3/7dof/urdf/gen3_macro.xacro" />
     <!-- Load the arm -->
     <xacro:load_arm

Commit message: Updating vision modules and adding yolo

File: ros2_kortex/kortex_description/robots/gen3.xacro (robot description, xacro)
@@ -4,5 +4,5 @@
     <xacro:arg name="arm" default="gen3" />
     <xacro:arg name="dof" default="7" />
-    <xacro:arg name="vision" default="false" />
+    <xacro:arg name="vision" default="true" />
     <xacro:arg name="robot_ip" default="192.168.11.11" />
     <xacro:arg name="username" default="admin" />
@@ -30,25 +30,29 @@
     <xacro:property name="initial_positions_file" default="$(arg initial_positions_file)"/>
     <link name="world">
-      <!-- Inertial properties -->
+    </link>
+    <link name="table">
       <inertial>
         <origin xyz="0 0 0" rpy="0 0 0" />
-        <mass value="1.0" /> <!-- Adjust mass as needed -->
+        <mass value="1.0" />
         <inertia ixx="0.1" ixy="0.0" ixz="0.0" iyy="0.1" iyz="0.0" izz="0.1" />
       </inertial>
-      <!-- Visual properties -->
       <visual>
         <origin xyz="0 0 0" rpy="0 0 0" />
         <geometry>
-          <box size="2 1 0.2" />
+          <box size="2 1 0.1" />
         </geometry>
       </visual>
-      <!-- Collision properties -->
       <collision>
         <origin xyz="0 0 0" rpy="0 0 0" />
         <geometry>
-          <box size="2 1 0.2" />
+          <box size="2 1 0.1" />
         </geometry>
       </collision>
     </link>
+  <joint name="table_joint" type="fixed">
+    <origin xyz="0.95 0 -0.08" rpy="0.0 0.0 0.0" />
+      <parent link="world"/>
+      <child link="table" />
+  </joint>
     <xacro:load_robot
         parent="world"

File: ros2_kortex/kortex_description/robots/kinova.urdf.xacro (robot description, xacro)
@@ -40,4 +40,6 @@
     <!-- World link -->
   <link name="world">
+  </link>
+  <link name="table">
     <inertial>
       <origin xyz="0 0 0" rpy="0 0 0" />
@@ -48,5 +50,5 @@
       <origin xyz="0 0 0" rpy="0 0 0" />
       <geometry>
-        <box size="2 1 0.2" />
+        <box size="2 1 0.1" />
       </geometry>
     </visual>
@@ -54,8 +56,13 @@
       <origin xyz="0 0 0" rpy="0 0 0" />
       <geometry>
-        <box size="2 1 0.2" />
+        <box size="2 1 0.1" />
       </geometry>
     </collision>
   </link>
+  <joint name="table_joint" type="fixed">
+    <origin xyz="0.95 0 -0.05" rpy="0.0 0.0 0.0" />
+      <parent link="world"/>
+      <child link="table" />
+  </joint>
   <xacro:load_robot
     parent="world"
