Commit message: Fixing the moveit config

File: ros2_kortex/kortex_moveit_config/kinova_gen3_7dof_robotiq_2f_85_moveit_config/config/gen3.ros2_control.xacro (robot description, xacro)
@@ -1,5 +1,5 @@
 <?xml version="1.0"?>
 <robot xmlns:xacro="http://www.ros.org/wiki/xacro">
-    <xacro:macro name="gen3_lite_ros2_control" params="name initial_positions_file">
+    <xacro:macro name="gen3_ros2_control" params="name initial_positions_file">
         <xacro:property name="initial_positions" value="${load_yaml(initial_positions_file)['initial_positions']}"/>
         <ros2_control name="${name}" type="system">
@@ -50,8 +50,15 @@
                 <state_interface name="velocity"/>
             </joint>
-            <joint name="right_finger_bottom_joint">
+            <joint name="joint_7">
                 <command_interface name="position"/>
                 <state_interface name="position">
-                  <param name="initial_value">${initial_positions['right_finger_bottom_joint']}</param>
+                  <param name="initial_value">${initial_positions['joint_7']}</param>
+                </state_interface>
+                <state_interface name="velocity"/>
+            </joint>
+            <joint name="robotiq_85_left_knuckle_joint">
+                <command_interface name="position"/>
+                <state_interface name="position">
+                  <param name="initial_value">${initial_positions['robotiq_85_left_knuckle_joint']}</param>
                 </state_interface>
                 <state_interface name="velocity"/>

File: test_saves/gen3.ros2_control.xacro (robot description, xacro)
@@ -1,5 +1,5 @@
 <?xml version="1.0"?>
 <robot xmlns:xacro="http://www.ros.org/wiki/xacro">
-    <xacro:macro name="gen3_lite_gen3_lite_2f_ros2_control" params="name initial_positions_file">
+    <xacro:macro name="gen3_ros2_control" params="name initial_positions_file">
         <xacro:property name="initial_positions" value="${load_yaml(initial_positions_file)['initial_positions']}"/>
         <ros2_control name="${name}" type="system">
@@ -50,8 +50,15 @@
                 <state_interface name="velocity"/>
             </joint>
-            <joint name="right_finger_bottom_joint">
+            <joint name="joint_7">
                 <command_interface name="position"/>
                 <state_interface name="position">
-                  <param name="initial_value">${initial_positions['right_finger_bottom_joint']}</param>
+                  <param name="initial_value">${initial_positions['joint_7']}</param>
+                </state_interface>
+                <state_interface name="velocity"/>
+            </joint>
+            <joint name="robotiq_85_left_knuckle_joint">
+                <command_interface name="position"/>
+                <state_interface name="position">
+                  <param name="initial_value">${initial_positions['robotiq_85_left_knuckle_joint']}</param>
                 </state_interface>
                 <state_interface name="velocity"/>
